Commit message: fixed error,add msg

File: rm_control/rm_description/urdf/common/swerve_drive.urdf.xacro (robot description, xacro)
@@ -1,55 +1,30 @@
 <robot xmlns:xacro="http://www.ros.org/wiki/xacro">
     <xacro:macro name="swerve_drive"
-                 params="prefix wheel_x_offset wheel_y_offset wheel_z_offset  connected_to reflect mirror">
+                 params="prefix wheel_x_offset wheel_y_offset wheel_z_offset  connected_to">
         <link name="${prefix}_pivot">
             <visual>
                 <origin xyz="0 0 0" rpy="0 0 0"/>
                 <geometry>
-                    <xacro:if value="${reflect == 1}">
-                        <mesh filename="package://rm_description/meshes/common/right_front_swerve_pivot.stl"
-                              scale="0.001 0.001 0.001"/>
-                    </xacro:if>
-                    <xacro:if value="${reflect == -1}">
-                        <mesh filename="package://rm_description/meshes/common/left_front_swerve_pivot.stl"
-                              scale="0.001 0.001 0.001"/>
-                    </xacro:if>
+                    <mesh filename="package://rm_description/meshes/common/swerve_pivot.stl"
+                          scale="0.001 0.001 0.001"/>
                 </geometry>
             </visual>
             <inertial>
-                <xacro:if value="${reflect == 1}">
                     <mass value="0.854"/>
                     <origin xyz="0.000054 0.008 0.00548" rpy="0 0 0"/>
                     <inertia ixx="6.711e-4" ixy="1.958e-9" ixz="-1.109e-6" iyy="6.703e-4" iyz="-1.095e-7"
                              izz="7.091e-4"/>
-                </xacro:if>
-                <xacro:if value="${reflect == -1}">
-                    <mass value="0.854"/>
-                    <origin xyz="0.000054 0.008 0.00548" rpy="0 0 0"/>
-                    <inertia ixx="6.711e-4" ixy="1.958e-9" ixz="-1.109e-6" iyy="6.703e-4" iyz="-1.095e-7"
-                             izz="7.091e-4"/>
-                </xacro:if>
             </inertial>
             <collision>
                 <origin xyz="0 0 0" rpy="0 0 0"/>
                 <geometry>
-                    <xacro:if value="${reflect == 1}">
-                        <mesh filename="package://rm_description/meshes/common/right_front_swerve_pivot.stl"
-                              scale="0.001 0.001 0.001"/>
-                    </xacro:if>
-                    <xacro:if value="${reflect == -1}">
-                        <mesh filename="package://rm_description/meshes/common/left_front_swerve_pivot.stl"
-                              scale="0.001 0.001 0.001"/>
-                    </xacro:if>
+                    <mesh filename="package://rm_description/meshes/common/swerve_pivot.stl"
+                          scale="0.001 0.001 0.001"/>
                 </geometry>
             </collision>
         </link>
-        <joint name="${prefix}_pivot_joint" type="continuous">
+        <joint name="${prefix}_pivot_joint" type="revolute">
             <axis xyz="0 0 1"/>
-            <xacro:if value="${mirror == 1}">
-                <origin xyz="${wheel_x_offset} ${wheel_y_offset} ${wheel_z_offset}" rpy="0 0 0"/>
-            </xacro:if>
-            <xacro:if value="${mirror == -1}">
-                <origin xyz="${wheel_x_offset} ${wheel_y_offset} ${wheel_z_offset}" rpy="0 0 ${pi}"/>
-            </xacro:if>
+            <origin xyz="${wheel_x_offset} ${wheel_y_offset} ${wheel_z_offset}" rpy="0 0 0"/>
             <parent link="${connected_to}"/>
             <child link="${prefix}_pivot"/>
@@ -77,5 +52,5 @@
             </collision>
         </link>
-        <joint name="${prefix}_wheel_joint" type="continuous">
+        <joint name="${prefix}_wheel_joint" type="revolute">
             <axis xyz="0 1 0"/>
             <origin xyz="0 0 -0.112" rpy="0 0 0"/>

File: rm_control/rm_description/urdf/engineer/arm.transmission.xacro (robot description, xacro)
@@ -6,9 +6,19 @@
             <type>transmission_interface/SimpleTransmission</type>
             <actuator name="joint1_motor">
-                <mechanicalReduction>71.75</mechanicalReduction>
+                <mechanicalReduction>3</mechanicalReduction>
             </actuator>
             <joint name="joint1">
                 <hardwareInterface>hardware_interface/EffortJointInterface</hardwareInterface>
-                <offset>2.068</offset>
+                <offset>0</offset>
+            </joint>
+        </transmission>
+        <transmission name="trans_joint2">
+            <type>transmission_interface/SimpleTransmission</type>
+            <actuator name="joint1_motor2">
+                <mechanicalReduction>3</mechanicalReduction>
+            </actuator>
+            <joint name="joint2">
+                <hardwareInterface>hardware_interface/EffortJointInterface</hardwareInterface>
+                <offset>0</offset>
             </joint>
         </transmission>
@@ -20,5 +30,5 @@
             <joint name="joint3">
                 <hardwareInterface>hardware_interface/EffortJointInterface</hardwareInterface>
-                <offset>-0.85</offset>
+                <offset>0</offset>
             </joint>
         </transmission>
@@ -26,9 +36,9 @@
             <type>transmission_interface/SimpleTransmission</type>
             <actuator name="joint4_motor">
-                <mechanicalReduction>-71.165</mechanicalReduction>
+                <mechanicalReduction>3</mechanicalReduction>
             </actuator>
             <joint name="joint4">
                 <hardwareInterface>hardware_interface/EffortJointInterface</hardwareInterface>
-                <offset>-0.334978036</offset>
+                <offset>0</offset>
             </joint>
         </transmission>
@@ -36,41 +46,31 @@
             <type>transmission_interface/SimpleTransmission</type>
             <actuator name="joint5_motor">
-                <mechanicalReduction>50.895</mechanicalReduction>
+                <mechanicalReduction>3</mechanicalReduction>
             </actuator>
             <joint name="joint5">
                 <hardwareInterface>hardware_interface/EffortJointInterface</hardwareInterface>
-                <offset>1.4378487</offset>
+                <offset>0</offset>
             </joint>
         </transmission>
-        <xacro:unless value="${simulation}">
-            <transmission name="trans_joint2">
-                <type>transmission_interface/DoubleActuatorTransmission</type>
-                <actuator name="joint2_left_motor">
-                    <role>actuator1</role>
-                    <mechanicalReduction>3</mechanicalReduction>
-                </actuator>
-                <actuator name="joint2_right_motor">
-                    <role>actuator2</role>
-                    <mechanicalReduction>-3</mechanicalReduction>
-                </actuator>
-                <joint name="joint2">
-                    <hardwareInterface>hardware_interface/EffortJointInterface</hardwareInterface>
-                    <offset>-2.391650</offset>
-                    <mechanicalReduction>1</mechanicalReduction>
-                </joint>
-            </transmission>
-        </xacro:unless>
-        <xacro:if value="${simulation}">
-            <transmission name="trans_joint2">
-                <type>transmission_interface/SimpleTransmission</type>
-                <actuator name="joint2_motor">
-                    <mechanicalReduction>-3</mechanicalReduction>
-                </actuator>
-                <joint name="joint2">
-                    <hardwareInterface>hardware_interface/EffortJointInterface</hardwareInterface>
-                    <offset>-2.3764</offset>
-                </joint>
-            </transmission>
-        </xacro:if>
+        <transmission name="trans_joint6">
+            <type>transmission_interface/SimpleTransmission</type>
+            <actuator name="joint6_motor">
+                <mechanicalReduction>3</mechanicalReduction>
+            </actuator>
+            <joint name="joint6">
+                <hardwareInterface>hardware_interface/EffortJointInterface</hardwareInterface>
+                <offset>0</offset>
+            </joint>
+        </transmission>
+        <transmission name="trans_joint7">
+            <type>transmission_interface/SimpleTransmission</type>
+            <actuator name="joint7_motor">
+                <mechanicalReduction>3</mechanicalReduction>
+            </actuator>
+            <joint name="joint7">
+                <hardwareInterface>hardware_interface/EffortJointInterface</hardwareInterface>
+                <offset>0</offset>
+            </joint>
+        </transmission>
     </xacro:macro>
 </robot>
